Commit message: Created gazebo_control to move robot in gazebo

File: description/robot.urdf.xacro (robot description, xacro)
@@ -2,3 +2,4 @@
 <robot xmlns:xacro="http://www.ros.org/wiki/xacro"  name="dynabot">
     <xacro:include filename="robot_core.xacro" />
+    <xacro:include filename="gazebo_control.xacro" />
 </robot>

File: description/robot_core.xacro (robot description, xacro)
@@ -44,4 +44,7 @@
         </xacro:inertial_box>
     </link>
+    <gazebo reference="chassis">
+        <material>Gazebo/White</material>
+    </gazebo>
     <!--LEFT WHEEL LINK-->
     <joint name="left_wheel_joint" type="continuous">
@@ -69,4 +72,7 @@
         </xacro:inertial_cylinder>
     </link>
+    <gazebo reference="left_wheel">
+        <material>Gazebo/Blue</material>
+    </gazebo>
     <!--RIGHT WHEEL LINK-->
     <joint name="right_wheel_joint" type="continuous">
@@ -94,4 +100,7 @@
         </xacro:inertial_cylinder>
     </link>
+    <gazebo reference="right_wheel">
+        <material>Gazebo/Blue</material>
+    </gazebo>
     <!--FRONT CASTER WHEEL LINK-->
     <joint name="front_caster_wheel_joint" type="fixed">
@@ -116,4 +125,9 @@
         </xacro:inertial_sphere>
     </link>
+    <gazebo reference="front_caster_wheel">
+        <material>Gazebo/Black</material>
+        <mu1 value="0.001" />
+        <mu2 value="0.001" />
+    </gazebo>
     <!--REAR CASTER WHEEL LINK-->
     <joint name="rear_caster_wheel_joint" type="fixed">
@@ -138,4 +152,9 @@
         </xacro:inertial_sphere>
     </link>
+    <gazebo reference="rear_caster_wheel">
+        <material>Gazebo/Black</material>
+        <mu1 value="0.001" />
+        <mu2 value="0.001" />
+    </gazebo>
     <!--BOTTOM FRAME-->
     <joint name="bottom_frame_joint" type="fixed">
@@ -162,4 +181,7 @@
         </xacro:inertial_box>
     </link>
+    <gazebo reference="bottom_frame">
+        <material>Gazebo/White</material>
+    </gazebo>
     <!--TOP FRAME-->
     <joint name="top_frame_joint" type="fixed">
@@ -186,4 +208,7 @@
         </xacro:inertial_box>
     </link>
+    <gazebo reference="top_frame">
+        <material>Gazebo/White</material>
+    </gazebo>
     <!--CAMERA-->
     <joint name="camera_joint" type="fixed">
@@ -210,4 +235,7 @@
         </xacro:inertial_box>
     </link>
+    <gazebo reference="camera_link">
+        <material>Gazebo/Red</material>
+    </gazebo>
     <!--GPS HOLDER + LIGHTS-->
     <joint name="gps_holder_joint" type="fixed">
@@ -234,4 +262,7 @@
         </xacro:inertial_cylinder>
     </link>
+    <gazebo reference="gps_holder_link">
+        <material>Gazebo/White</material>
+    </gazebo>
     <!--GPS-->
     <joint name="gps_joint" type="fixed">
@@ -258,4 +289,7 @@
         </xacro:inertial_box>
     </link>
+    <gazebo reference="gps_link">
+        <material>Gazebo/Red</material>
+    </gazebo>
     <!--IMU-->
     <joint name="imu_joint" type="fixed">
@@ -282,3 +316,6 @@
         </xacro:inertial_box>
     </link>
+    <gazebo reference="imu_link">
+        <material>Gazebo/Red</material>
+    </gazebo>
 </robot>

Commit message: Added ros2_control and started to make it work for real robot. Still have to add more ros2_control stuff.

File: description/robot.urdf.xacro (robot description, xacro)
@@ -1,5 +1,15 @@
 <?xml version="1.0"?>
 <robot xmlns:xacro="http://www.ros.org/wiki/xacro"  name="dynabot">
+    <xacro:arg name="use_ros2_control" default="true"/>
+    <xacro:arg name="sim_mode" default="true"/>
     <xacro:include filename="robot_core.xacro" />
-    <xacro:include filename="gazebo_control.xacro" />
+    <xacro:if value="$(arg use_ros2_control)">
+        <xacro:include filename="ros2_control.xacro" />
+    </xacro:if>
+    <xacro:unless value="$(arg use_ros2_control)">
+        <xacro:include filename="gazebo_control.xacro" />
+    </xacro:unless>
+    <xacro:include filename="lidar.xacro" />
+    <!-- <xacro:include filename="camera.xacro" /> -->
+    <!-- <xacro:include filename="depth_camera.xacro" /> -->
 </robot>

File: description/robot_core.xacro (robot description, xacro)
@@ -65,5 +65,5 @@
             <origin xyz="0 0 0.0681" />
             <geometry>
-                <cylinder radius="0.202" length=".1362" />
+                <sphere radius="0.202" />
             </geometry>
         </collision>
@@ -93,5 +93,5 @@
             <origin xyz="0 0 0.0681" />
             <geometry>
-                <cylinder radius="0.202" length=".1362" />
+                <sphere radius="0.202" />
             </geometry>
         </collision>
