Commit message: Added regular camera for simulation

File: description/lidar.xacro (robot description, xacro)
@@ -30,5 +30,5 @@
         <sensor name="laser" type="ray">
             <pose>0 0 0 0 0 0</pose>
-            <visualize>true</visualize>
+            <visualize>false</visualize>
             <update_rate>10</update_rate>
             <ray>

File: description/robot.urdf.xacro (robot description, xacro)
@@ -11,5 +11,5 @@
     </xacro:unless>
     <xacro:include filename="lidar.xacro" />
-    <!-- <xacro:include filename="camera.xacro" /> -->
+    <xacro:include filename="camera.xacro" />
     <!-- <xacro:include filename="depth_camera.xacro" /> -->
 </robot>

File: description/robot_core.xacro (robot description, xacro)
@@ -211,31 +211,4 @@
         <material>Gazebo/White</material>
     </gazebo>
-    <!--CAMERA-->
-    <joint name="camera_joint" type="fixed">
-        <parent link="bottom_frame" />
-        <child link="camera_link" />
-        <origin xyz="0.6947 0 0.2858" />
-    </joint>
-    <link name="camera_link">
-        <visual>
-            <origin xyz="-0.01755 0 0" />
-            <geometry>
-                <box size="0.0351 0.1143 0.0254" />
-            </geometry>
-            <material name="red" />
-        </visual>
-        <collision>
-            <origin xyz="-0.01755 0 0" />
-            <geometry>
-                <box size="0.0351 0.1143 0.0254"  />
-            </geometry>
-        </collision>
-        <xacro:inertial_box mass="0.13" x="0.0351" y="0.1143" z="0.0254">
-            <origin xyz="-0.01755 0 0" rpy="0 0 0" />
-        </xacro:inertial_box>
-    </link>
-    <gazebo reference="camera_link">
-        <material>Gazebo/Red</material>
-    </gazebo>
     <!--GPS HOLDER + LIGHTS-->
     <joint name="gps_holder_joint" type="fixed">

Commit message: Updated dynabot to work with dynabot-ros

File: description/lidar.xacro (robot description, xacro)
@@ -4,8 +4,8 @@
     <joint name="laser_joint" type="fixed">
         <parent link="bottom_frame" />
-        <child link="laser_frame" />
+        <child link="laser" />
         <origin xyz="0.73915 0 0.1336" />
     </joint>
-    <link name="laser_frame">
+    <link name="laser">
         <visual>
             <origin xyz="-0.039775 0 -0.03715" />

File: description/ros2_control.xacro (robot description, xacro)
@@ -4,5 +4,5 @@
         <ros2_control name="RealRobot" type="system">
             <hardware>
-                <plugin>dynabot_control/DiffDriveDynabotHardware</plugin>
+                <plugin>dynabot_hardware/DynabotSystemHardware</plugin>
                 <param name="serial_port">/dev/ttyACM0</param>
                 <param name="wheel_radius">0.202</param>
